File: ShiftyBoi.kicad_sch (KiCad schematic)
At the start: 18 parts, among them J1 Screw_Terminal_01x08, J2 Screw_Terminal_01x08, J3 Screw_Terminal_01x08, J4 Screw_Terminal_01x08, J5 Screw_Terminal_01x08, J6 PROG, J7 Barrel_Jack_MountingPin, U1 ESP-12F, U2 74HC595, U3 74HC595, U4 74HC595, U5 74HC595, U6 AMS1117-3.3

Commit message: Final PCB Layout
Parts:
- C1: value C -> 10uf; LCSC Part (none) -> C13585
- C2: value C -> 100uf; LCSC Part (none) -> C15008
- R1: LCSC Part (none) -> C25900
- R2, R3: LCSC Part (none) -> C25744
- U1: LCSC Part (none) -> C82891
- U2, U3, U5: LCSC Part (none) -> C5947
- U4: C5947 (none) -> LCSC Part
- U6: LCSC Part (none) -> C6186
Changed lines of the file:
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@@
+      (effects (font (size 1.27 1.27)) hide)
+    )
+    (property "LCSC Part" "C5947" (at 86.36 135.89 0)
       (effects (font (size 1.27 1.27)) hide)
     )
@@
       (effects (font (size 1.27 1.27)) hide)
     )
+    (property "LCSC Part" "C6186" (at 102.87 175.26 0)
+      (effects (font (size 1.27 1.27)) hide)
+    )
     (pin "1")
     (pin "2")
@@
       (effects (font (size 1.27 1.27)) hide)
     )
+    (property "LCSC Part" "C25744" (at 87.63 80.01 0)
+      (effects (font (size 1.27 1.27)) hide)
+    )
     (pin "1")
     (pin "2")
@@
       (effects (font (size 1.27 1.27)) (justify left))
     )
-    (property "Value" "C" (at 116.84 184.785 0)
+    (property "Value" "100uf" (at 116.84 184.785 0)
       (effects (font (size 1.27 1.27)) (justify left))
     )
@@
       (effects (font (size 1.27 1.27)) hide)
     )
+    (property "LCSC Part" "C15008" (at 113.03 182.88 0)
+      (effects (font (size 1.27 1.27)) hide)
+    )
     (pin "1")
     (pin "2")
@@
       (effects (font (size 1.27 1.27)) (justify left))
     )
-    (property "Value" "C" (at 96.52 184.785 0)
+    (property "Value" "10uf" (at 96.52 184.785 0)
       (effects (font (size 1.27 1.27)) (justify left))
     )
@@
     )
     (property "Datasheet" "~" (at 92.71 182.88 0)
+      (effects (font (size 1.27 1.27)) hide)
+    )
+    (property "LCSC Part" "C13585" (at 92.71 182.88 0)
       (effects (font (size 1.27 1.27)) hide)
     )
@@
     )
     (property "Datasheet" "http://wiki.ai-thinker.com/_media/esp8266/esp8266_series_modules_user_manual_v1.1.pdf" (at 55.88 64.77 0)
+      (effects (font (size 1.27 1.27)) hide)
+    )
+    (property "LCSC Part" "C82891" (at 64.77 67.31 0)
       (effects (font (size 1.27 1.27)) hide)
     )
@@
       (effects (font (size 1.27 1.27)) hide)
     )
+    (property "LCSC Part" "C25900" (at 48.26 46.99 0)
+      (effects (font (size 1.27 1.27)) hide)
+    )
     (pin "1")
     (pin "2")
@@
     )
     (property "Datasheet" "http://www.ti.com/lit/ds/symlink/sn74hc595.pdf" (at 167.64 135.89 0)
+      (effects (font (size 1.27 1.27)) hide)
+    )
+    (property "LCSC Part" "C5947" (at 167.64 135.89 0)
       (effects (font (size 1.27 1.27)) hide)
     )
@@
       (effects (font (size 1.27 1.27)) hide)
     )
+    (property "C5947" "LCSC Part" (at 127 135.89 0)
+      (effects (font (size 1.27 1.27)) hide)
+    )
     (pin "1")
     (pin "10")
@@
       (effects (font (size 1.27 1.27)) hide)
     )
+    (property "LCSC Part" "C25744" (at 81.28 46.99 0)
+      (effects (font (size 1.27 1.27)) hide)
+    )
     (pin "1")
     (pin "2")
@@
       (effects (font (size 1.27 1.27)) hide)
     )
+    (property "LCSC Part" "C5947" (at 45.72 135.89 0)
+      (effects (font (size 1.27 1.27)) hide)
+    )
