File: drivers.kicad_sch (KiCad schematic)
At the start: 96 parts, among them Q1 AO3400A

Commit message: Final PCB Layout
Parts:
- Q1: LCSC Part (none) -> C20917
- R1: LCSC Part (none) -> C11702
- R2: LCSC Part (none) -> C25744
